File: pcb/2_POE.kicad_sch (KiCad schematic)
At the start: 36 parts, among them J1 RJ45_LED_Shielded, U2 DP1435-12V, U3 RTL8201F-VB-CG

Commit message: review version
Parts:
- added C45: 330u / 25V, Capacitor_SMD:CP_Elec_8x10.5, symbol Device:C_Polarized
- added C46: 47uF, Capacitor_SMD:C_1206_3216Metric, symbol Device:C
- added L5: 3.3µH / 3.1A, Inductor_SMD:L_Changjiang_FNR5030S, symbol Device:L
- C10, C12, C9: footprint Capacitor_SMD:C_0805_2012Metric -> Capacitor_SMD:C_1206_3216Metric; LCSC C16780 -> C22367835
- C4: value 1nF -> 1nF / 2KV
- C5, C6, C7, C8: value 10nF -> 10nF / 100V; LCSC C57112 -> C43253
- R14: value 2.49kΩ -> 2K49
- R15, R18: value 220Ω -> 220
- R16, R17: value 10kΩ -> 2K49; LCSC C25804 -> C22908
Connections:
- net +12V_POE: now also C46.2, L5.2; no longer U2.6 (+12V)
- net GND: now also C45.2, C46.1
- new net: C45.1, L5.1, U2.6 (+12V)
Other:
- note added: "COL auf TP oder LED"
- note added: "PU = RMII"
- note added: "TXD+ und TXD- muss TXD[0] und TXD[1] das Gleiche bei RXD"
- moved on the sheet: C18

Commit message: remove third pcb and more flash
Parts:
- C11: LCSC C57112 -> C43253
- R14, R16, R17: value 2K49 -> 2.49Ω
- R15, R18: value 220 -> 220Ω
Connections:
- net EMAC_RXD+ renamed EMAC_RXD0
- net EMAC_RXD- renamed EMAC_RXD1
- net EMAC_TXD+ renamed EMAC_TXD0
- net EMAC_TXD- renamed EMAC_TXD1
Other:
- note removed: "COL auf TP oder LED"
- note removed: "TXD+ und TXD- muss TXD[0] und TXD[1] das Gleiche bei RXD"
Changed lines of the file:
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@@
 		)
 	)
-	(text "TXD+ und TXD- muss TXD[0] und TXD[1]\ndas Gleiche bei RXD"
-		(exclude_from_sim no)
-		(at 297.18 149.225 90)
-		(effects
-			(font
-				(size 1.27 1.27)
-			)
-		)
-	)
-	(text "COL auf TP oder LED"
-		(exclude_from_sim no)
-		(at 259.08 79.375 90)
-		(effects
-			(font
-				(size 1.27 1.27)
-			)
-		)
-	)
 	(label "RCT"
 		(at 143.51 121.92 0)
@@
 		)
 	)
-	(hierarchical_label "EMAC_RXD+"
+	(hierarchical_label "EMAC_RXD0"
 		(shape output)
 		(at 246.38 163.83 270)
@@
 		)
 	)
-	(hierarchical_label "EMAC_TXD+"
+	(hierarchical_label "EMAC_TXD0"
 		(shape input)
 		(at 264.16 163.83 270)
@@
 		)
 	)
-	(hierarchical_label "EMAC_RXD-"
+	(hierarchical_label "EMAC_RXD1"
 		(shape output)
 		(at 248.92 163.83 270)
@@
 		)
 	)
-	(hierarchical_label "EMAC_TXD-"
+	(hierarchical_label "EMAC_TXD1"
 		(shape input)
 		(at 295.91 132.08 0)
@@
 		)
 		(property "Value" "GND"
-			(at 53.34 115.57 0)
+			(at 50.8 111.7599 0)
 			(effects
 				(font
 					(size 1.27 1.27)
 				)
+				(justify left)
 			)
 		)
@@
 		(on_board yes)
 		(dnp no)
+		(fields_autoplaced yes)
 		(property "Reference" "C10"
-			(at 140.97 32.385 90)
+			(at 140.97 27.94 90)
 			(effects
 				(font
@@
 		)
 		(property "Value" "47uF"
-			(at 144.78 34.29 90)
+			(at 140.97 30.48 90)
 			(effects
 				(font
@@
 		(on_board yes)
 		(dnp no)
+		(fields_autoplaced yes)
 		(property "Reference" "R18"
-			(at 331.47 78.105 90)
+			(at 332.74 73.66 90)
 			(effects
 				(font
@@
 			)
 		)
-		(property "Value" "220"
-			(at 332.74 80.01 90)
+		(property "Value" "220Ω"
+			(at 332.74 76.2 90)
 			(effects
 				(font
@@
 		(on_board yes)
 		(dnp no)
+		(fields_autoplaced yes)
 		(property "Reference" "R16"
-			(at 331.47 61.595 90)
+			(at 332.74 57.15 90)
 			(effects
 				(font
@@
 			)
 		)
-		(property "Value" "2K49"
-			(at 332.74 63.5 90)
+		(property "Value" "2.49Ω"
+			(at 332.74 59.69 90)
 			(effects
 				(font
@@
 		(on_board yes)
 		(dnp no)
+		(fields_autoplaced yes)
 		(property "Reference" "R17"
-			(at 331.47 69.215 90)
+			(at 332.74 64.77 90)
 			(effects
 				(font
@@
 			)
 		)
-		(property "Value" "2K49"
-			(at 332.74 71.12 90)
+		(property "Value" "2.49Ω"
+			(at 332.74 67.31 90)
 			(effects
 				(font
@@
 		(on_board yes)
 		(dnp no)
+		(fields_autoplaced yes)
 		(property "Reference" "R15"
-			(at 331.47 52.705 90)
+			(at 332.74 48.26 90)
 			(effects
 				(font
@@
 			)
 		)
-		(property "Value" "220"
-			(at 332.74 54.61 90)
+		(property "Value" "220Ω"
+			(at 332.74 50.8 90)
 			(effects
 				(font
@@
 			)
 		)
-		(property "LCSC" "C57112"
+		(property "LCSC" "C43253"
 			(at 154.94 140.97 0)
 			(effects
@@
 		(on_board yes)
 		(dnp no)
+		(fields_autoplaced yes)
 		(property "Reference" "C9"
-			(at 140.97 22.225 90)
+			(at 140.97 17.78 90)
 			(effects
 				(font
@@
 		)
 		(property "Value" "47uF"
-			(at 144.78 24.13 90)
+			(at 140.97 20.32 90)
 			(effects
 				(font
@@
 			)
 		)
-		(property "Value" "2K49"
+		(property "Value" "2.49Ω"
 			(at 224.79 39.3699 0)
 			(effects
@@
 		)
 		(instances
-			(project ""
+			(project "Lichtstab"
 				(path "/e085f17c-3357-4281-ab9e-eebcecacdfc5/f0684335-54fe-4c40-868c-eb2ee3b6696b"
 					(reference "L5")
@@
 		(fields_autoplaced yes)
 		(property "Reference" "C45"
-			(at 102.235 242.9509 0)
+			(at 102.87 242.9509 0)
 			(effects
 				(font
@@
 		)
 		(property "Value" "330u / 25V"
-			(at 102.235 245.4909 0)
+			(at 102.87 245.4909 0)
 			(effects
 				(font
@@
 		)
 		(instances
-			(project ""
+			(project "Lichtstab"
 				(path "/e085f17c-3357-4281-ab9e-eebcecacdfc5/f0684335-54fe-4c40-868c-eb2ee3b6696b"
 					(reference "C45")
